File: hw/pod/draft_r1/pod_r1_placed.kicad_pcb (KiCad board)
At the start: 4 copper layers, 34 x 13 mm, 73 parts, among them J1 TestPoint_Pad_D1.0mm, J10 TestPoint_Pad_D1.0mm, J11 TestPoint_Pad_D1.0mm, J12 TestPoint_Pad_D1.0mm, J2 TestPoint_Pad_D1.0mm, J3 TestPoint_Pad_D1.0mm, J4 WirePad_1.0x2.0mm, J5 TestPoint_Pad_D1.0mm, J7 TestPoint_Pad_D1.0mm, J8 TestPoint_Pad_D1.0mm, J9 TestPoint_Pad_D1.0mm, Q1 Nexperia_SOT1216_DFN1010B-6, Q2 Nexperia_SOT1216_DFN1010B-6, SW1 SW-SMD_4P-L3.0-W2.6-P1.85-LS3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, U1 QFN-48-1EP_7x7mm_P0.5mm_EP5.6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, U2 Knowles_LGA-5_3.5x2.65mm, U3 DSBGA-8_L1.6-W0.9-R2-C4-P0.40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, U4 X2SON-4_L1.0-W1.0-P0.65-TL-EP, U6 SOT-553-5_L1.6-W1.2-P0.50-LS1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, Y1 FC-135R_L3.2-W1.5

Commit message: Rev G (ECR-0017, owner O24): C8/C9 back to 10 V-rated 2.2 uF C107369 (ST DS13737 Rev 10 p.153); D6 TPD1E10B06 ESD at the exposed CC contact J12 (same part/BOM line as D5)
- gen.py Rev G: 53 placed parts, 30 BOM lines, ERC 0; bom_check identity + part_heights for C107369
- board re-placed + routed (D6 on B behind J12, one via): 694 tracks, 118 vias, 1 unconnected (I2C_SDA, router
  variance), DRC 19 courtyard + 1 clearance 0.0892 vs 0.09 mm (router rounding); Phase-2 board supersedes it
- schematic pages regenerated (D6 on the dock sheet, Rev G title): connectivity PASS, 195 memberships
- tracker: new relations R-SMPS-BOARD, R-CLOCK-BOARD, R-UI-BOARD (miniaturization MZG-15 blind spot); all reviewed,
  0 suspect / 0 stale; docs updated (sub-processing issue 1 closed, sub-dock-usb F15, reg-board route, 00-whole counts)
- interfaces.py self-test: the clamp-band victim skips test pads (exempt by rule; the re-placement put TP7 first)

Co-Authored-By: Claude Opus 5.5 <noreply@anthropic.com>
Claude-Session: https://claude.ai/code/session_01Wg997D6KFs8bxoAH56jZZJ
Parts:
- added D6: X1SON-2_L1.0-W0.6-P0.65-BI-1, X1SON-2_L1.0-W0.6-P0.65-BI-1, B.Cu at (32.6, 6.20)
Routing:
- net GND: track 28.6 -> 29.1 mm, vias 45 -> 46
