File: hw/pod/sch/dock.kicad_sch (KiCad schematic)
At the start: 12 parts, among them J10 D+, J11 D-, J12 CC, J3 VBUS, J4 GND, U6 TPD2E2U06DRLR

Commit message: Rev G (ECR-0017, owner O24): C8/C9 back to 10 V-rated 2.2 uF C107369 (ST DS13737 Rev 10 p.153); D6 TPD1E10B06 ESD at the exposed CC contact J12 (same part/BOM line as D5)
- gen.py Rev G: 53 placed parts, 30 BOM lines, ERC 0; bom_check identity + part_heights for C107369
- board re-placed + routed (D6 on B behind J12, one via): 694 tracks, 118 vias, 1 unconnected (I2C_SDA, router
  variance), DRC 19 courtyard + 1 clearance 0.0892 vs 0.09 mm (router rounding); Phase-2 board supersedes it
- schematic pages regenerated (D6 on the dock sheet, Rev G title): connectivity PASS, 195 memberships
- tracker: new relations R-SMPS-BOARD, R-CLOCK-BOARD, R-UI-BOARD (miniaturization MZG-15 blind spot); all reviewed,
  0 suspect / 0 stale; docs updated (sub-processing issue 1 closed, sub-dock-usb F15, reg-board route, 00-whole counts)
- interfaces.py self-test: the clamp-band victim skips test pads (exempt by rule; the re-placement put TP7 first)

Co-Authored-By: Claude Opus 5.5 <noreply@anthropic.com>
Claude-Session: https://claude.ai/code/session_01Wg997D6KFs8bxoAH56jZZJ
Parts:
- added D6: TPD1E10B06DPYR, lcsc:X1SON-2_L1.0-W0.6-P0.65-BI-1, symbol lcsc:TPD1E10B06DPYR
Connections:
- net CC: now also D6.1
- net GND: now also D6.2
Other:
- title: Pod board Rev F: Dock and USB protection -> Pod board Rev G: Dock and USB protection
Changed lines of the file:
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@@
 	(paper "A4")
 	(title_block
-		(title "Pod board Rev F: Dock and USB protection")
+		(title "Pod board Rev G: Dock and USB protection")
 		(date "2026-10-02")
-		(rev "F")
+		(rev "G")
 		(company "Stereo Ultrasound")
 		(comment 1 "Generated by hw/pod/sch.py from hw/pod/pod.net (gen.py). Do not edit by hand.")
@@
 	(wire
 		(pts
+			(xy 43.18 147.32)
+			(xy 25.4 147.32)
+		)
+		(stroke
+			(width 0)
+			(type default)
+		)
+	)
+	(wire
+		(pts
+			(xy 55.88 148.59)
+			(xy 55.88 147.32)
+		)
+		(stroke
+			(width 0)
+			(type default)
+		)
+	)
+	(wire
+		(pts
+			(xy 55.88 147.32)
+			(xy 43.18 147.32)
+		)
+		(stroke
+			(width 0)
+			(type default)
+		)
+	)
+	(wire
+		(pts
 			(xy 50.8 54.61)
 			(xy 50.8 50.8)
@@
 			(xy 109.22 50.8)
 			(xy 91.44 50.8)
-		)
-		(stroke
-			(width 0)
-			(type default)
-		)
-	)
-	(wire
-		(pts
-			(xy 43.18 147.32)
-			(xy 25.4 147.32)
 		)
 		(stroke
@@
 		)
 	)
+	(text_box "SPARK GUARD  D6\nThe same guard on the CC contact, the last exposed contact that had none (Rev G)."
+		(exclude_from_sim no)
+		(at 139.7 125.73 0)
+		(size 76.2 12.7)
+		(margins 0.9525 0.9525 0.9525 0.9525)
+		(stroke
+			(width 0)
+			(type default)
+		)
+		(fill
+			(type color)
+			(color 255 248 225 1)
+		)
+		(effects
+			(font
+				(size 1.524 1.524)
+			)
+			(justify left top)
+		)
+	)
 	(symbol
 		(lib_id "Connector:TestPoint")
@@
 	)
 	(symbol
+		(lib_id "lcsc:TPD1E10B06DPYR")
+		(at 55.88 153.67 270)
+		(unit 1)
+		(exclude_from_sim no)
+		(in_bom yes)
+		(on_board yes)
+		(dnp no)
+		(property "Reference" "D6"
+			(at 60.22 153.07 90)
+			(effects
+				(font
+					(size 1.27 1.27)
+				)
+			)
+		)
+		(property "Value" "TPD1E10B06DPYR"
+			(at 66.52 155.57 90)
+			(effects
+				(font
+					(size 1.27 1.27)
+				)
+			)
+		)
+		(property "Footprint" "lcsc:X1SON-2_L1.0-W0.6-P0.65-BI-1"
+			(at 55.88 153.67 90)
+			(effects
+				(font
+					(size 1.27 1.27)
+				)
+				(hide yes)
+			)
+		)
+		(property "Datasheet" ""
+			(at 55.88 153.67 90)
+			(effects
+				(font
+					(size 1.27 1.27)
+				)
+				(hide yes)
+			)
+		)
+		(property "LCSC" "C48260"
+			(at 55.88 153.67 0)
+			(effects
+				(font
+					(size 1.27 1.27)
+				)
+				(hide yes)
+			)
+		)
+		(pin "2"
+		)
+		(pin "1"
+		)
+		(instances
+			(project "pod"
+				(path "/46f56cb9-40b8-53c9-9ea1-5c731f397bba/a2aaa97b-438e-5f97-8bd8-ad6e32f4aee8"
+					(reference "D6")
+					(unit 1)
+				)
+			)
+		)
+	)
+	(symbol
 		(lib_id "power:VCC")
 		(at 25.4 177.8 0)
@@
 	)
 	(symbol
+		(lib_id "power:GND")
+		(at 55.88 158.75 0)
+		(unit 1)
+		(exclude_from_sim no)
+		(in_bom no)
+		(on_board yes)
+		(dnp no)
+		(property "Reference" "#PWR009"
+			(at 55.88 158.75 0)
+			(effects
+				(font
+					(size 1.27 1.27)
+				)
+				(hide yes)
+			)
+		)
+		(property "Value" "GND"
+			(at 55.88 162.56 0)
+			(effects
+				(font
+					(size 1.27 1.27)
+				)
+				(hide yes)
+			)
+		)
+		(property "Footprint" ""
+			(at 55.88 158.75 0)
+			(effects
+				(font
+					(size 1.27 1.27)
+				)
+				(hide yes)
+			)
+		)
+		(property "Datasheet" ""
+			(at 55.88 158.75 0)
+			(effects
+				(font
+					(size 1.27 1.27)
+				)
+				(hide yes)
+			)
+		)
+		(pin "1"
+		)
+		(instances
+			(project "pod"
+				(path "/46f56cb9-40b8-53c9-9ea1-5c731f397bba/a2aaa97b-438e-5f97-8bd8-ad6e32f4aee8"
+					(reference "#PWR009")
+					(unit 1)
+				)
+			)
+		)
+	)
+	(symbol
 		(lib_id "power:VCC")
 		(at 50.8 48.26 0)
@@
 		(on_board yes)
 		(dnp no)
-		(property "Reference" "#PWR009"
+		(property "Reference" "#PWR010"
 			(at 50.8 48.26 0)
 			(effects
@@
 			(project "pod"
 				(path "/46f56cb9-40b8-53c9-9ea1-5c731f397bba/a2aaa97b-438e-5f97-8bd8-ad6e32f4aee8"
-					(reference "#PWR009")
+					(reference "#PWR010")
 					(unit 1)
 				)
@@
 		(on_board yes)
 		(dnp no)
-		(property "Reference" "#PWR010"
+		(property "Reference" "#PWR011"
 			(at 91.44 48.26 0)
 			(effects
@@
 			(project "pod"
 				(path "/46f56cb9-40b8-53c9-9ea1-5c731f397bba/a2aaa97b-438e-5f97-8bd8-ad6e32f4aee8"
-					(reference "#PWR010")
-					(unit 1)
-				)
+					(reference "#PWR011")
+					(unit 1)
+				)
