File: hw/pod/sch/mic.kicad_sch (KiCad schematic)
At the start: 2 parts, among them U2 SPH0641LU4H-1

Commit message: Rev G (ECR-0017, owner O24): C8/C9 back to 10 V-rated 2.2 uF C107369 (ST DS13737 Rev 10 p.153); D6 TPD1E10B06 ESD at the exposed CC contact J12 (same part/BOM line as D5)
- gen.py Rev G: 53 placed parts, 30 BOM lines, ERC 0; bom_check identity + part_heights for C107369
- board re-placed + routed (D6 on B behind J12, one via): 694 tracks, 118 vias, 1 unconnected (I2C_SDA, router
  variance), DRC 19 courtyard + 1 clearance 0.0892 vs 0.09 mm (router rounding); Phase-2 board supersedes it
- schematic pages regenerated (D6 on the dock sheet, Rev G title): connectivity PASS, 195 memberships
- tracker: new relations R-SMPS-BOARD, R-CLOCK-BOARD, R-UI-BOARD (miniaturization MZG-15 blind spot); all reviewed,
  0 suspect / 0 stale; docs updated (sub-processing issue 1 closed, sub-dock-usb F15, reg-board route, 00-whole counts)
- interfaces.py self-test: the clamp-band victim skips test pads (exempt by rule; the re-placement put TP7 first)

Co-Authored-By: Claude Opus 5.5 <noreply@anthropic.com>
Claude-Session: https://claude.ai/code/session_01Wg997D6KFs8bxoAH56jZZJ
Other:
- title: Pod board Rev F: Microphone -> Pod board Rev G: Microphone
Changed lines of the file:
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@@
 	(paper "A4")
 	(title_block
-		(title "Pod board Rev F: Microphone")
+		(title "Pod board Rev G: Microphone")
 		(date "2026-10-02")
-		(rev "F")
+		(rev "G")
 		(company "Stereo Ultrasound")
 		(comment 1 "Generated by hw/pod/sch.py from hw/pod/pod.net (gen.py). Do not edit by hand.")
@@
 		(on_board yes)
 		(dnp no)
-		(property "Reference" "#PWR074"
+		(property "Reference" "#PWR075"
 			(at 88.9 73.66 90)
 			(effects
@@
 		(property "Datasheet" ""
 			(at 88.9 73.66 90)
-			(effects
-				(font
-					(size 1.27 1.27)
-				)
-				(hide yes)
-			)
-		)
-		(pin "1"
-		)
-		(instances
-			(project "pod"
-				(path "/46f56cb9-40b8-53c9-9ea1-5c731f397bba/253b1d4d-845e-5bbb-b17c-2d22e1c4b6f2"
-					(reference "#PWR074")
-					(unit 1)
-				)
-			)
-		)
-	)
-	(symbol
-		(lib_id "power:GND")
-		(at 76.2 83.82 0)
-		(unit 1)
-		(exclude_from_sim no)
-		(in_bom no)
-		(on_board yes)
-		(dnp no)
-		(property "Reference" "#PWR075"
-			(at 76.2 83.82 0)
-			(effects
-				(font
-					(size 1.27 1.27)
-				)
-				(hide yes)
-			)
-		)
-		(property "Value" "GND"
-			(at 76.2 87.63 0)
-			(effects
-				(font
-					(size 1.27 1.27)
-				)
-				(hide yes)
-			)
-		)
-		(property "Footprint" ""
-			(at 76.2 83.82 0)
-			(effects
-				(font
-					(size 1.27 1.27)
-				)
-				(hide yes)
-			)
-		)
-		(property "Datasheet" ""
-			(at 76.2 83.82 0)
 			(effects
 				(font
@@
 	(symbol
 		(lib_id "power:GND")
-		(at 55.88 80.01 0)
+		(at 76.2 83.82 0)
 		(unit 1)
 		(exclude_from_sim no)
@@
 		(dnp no)
 		(property "Reference" "#PWR076"
-			(at 55.88 80.01 0)
+			(at 76.2 83.82 0)
 			(effects
 				(font
@@
 		)
 		(property "Value" "GND"
-			(at 55.88 83.82 0)
+			(at 76.2 87.63 0)
 			(effects
 				(font
@@
 		)
 		(property "Footprint" ""
-			(at 55.88 80.01 0)
+			(at 76.2 83.82 0)
 			(effects
 				(font
@@
 		)
 		(property "Datasheet" ""
-			(at 55.88 80.01 0)
+			(at 76.2 83.82 0)
 			(effects
 				(font
@@
 	)
 	(symbol
+		(lib_id "power:GND")
+		(at 55.88 80.01 0)
+		(unit 1)
+		(exclude_from_sim no)
+		(in_bom no)
+		(on_board yes)
+		(dnp no)
+		(property "Reference" "#PWR077"
+			(at 55.88 80.01 0)
+			(effects
+				(font
+					(size 1.27 1.27)
+				)
+				(hide yes)
+			)
+		)
+		(property "Value" "GND"
+			(at 55.88 83.82 0)
+			(effects
+				(font
+					(size 1.27 1.27)
+				)
+				(hide yes)
+			)
+		)
+		(property "Footprint" ""
+			(at 55.88 80.01 0)
+			(effects
+				(font
+					(size 1.27 1.27)
+				)
+				(hide yes)
+			)
+		)
+		(property "Datasheet" ""
+			(at 55.88 80.01 0)
+			(effects
+				(font
+					(size 1.27 1.27)
+				)
+				(hide yes)
+			)
+		)
+		(pin "1"
+		)
+		(instances
+			(project "pod"
+				(path "/46f56cb9-40b8-53c9-9ea1-5c731f397bba/253b1d4d-845e-5bbb-b17c-2d22e1c4b6f2"
+					(reference "#PWR077")
+					(unit 1)
+				)
+			)
+		)
+	)
+	(symbol
 		(lib_id "power:PWR_FLAG")
 		(at 76.2 66.04 0)
@@
 		(on_board yes)
 		(dnp no)
-		(property "Reference" "#FLG077"
+		(property "Reference" "#FLG078"
 			(at 76.2 66.04 0)
 			(effects
@@
 			(project "pod"
 				(path "/46f56cb9-40b8-53c9-9ea1-5c731f397bba/253b1d4d-845e-5bbb-b17c-2d22e1c4b6f2"
-					(reference "#FLG077")
+					(reference "#FLG078")
 					(unit 1)
 				)
