File: hw/pod/sch/output.kicad_sch (KiCad schematic)
At the start: 15 parts, among them J1 XDCR_A, J2 XDCR_B, J7 LED+, J8 LED-, Q1 PMCXB290UE, Q2 PMCXB290UE

Commit message: Rev G (ECR-0017, owner O24): C8/C9 back to 10 V-rated 2.2 uF C107369 (ST DS13737 Rev 10 p.153); D6 TPD1E10B06 ESD at the exposed CC contact J12 (same part/BOM line as D5)
- gen.py Rev G: 53 placed parts, 30 BOM lines, ERC 0; bom_check identity + part_heights for C107369
- board re-placed + routed (D6 on B behind J12, one via): 694 tracks, 118 vias, 1 unconnected (I2C_SDA, router
  variance), DRC 19 courtyard + 1 clearance 0.0892 vs 0.09 mm (router rounding); Phase-2 board supersedes it
- schematic pages regenerated (D6 on the dock sheet, Rev G title): connectivity PASS, 195 memberships
- tracker: new relations R-SMPS-BOARD, R-CLOCK-BOARD, R-UI-BOARD (miniaturization MZG-15 blind spot); all reviewed,
  0 suspect / 0 stale; docs updated (sub-processing issue 1 closed, sub-dock-usb F15, reg-board route, 00-whole counts)
- interfaces.py self-test: the clamp-band victim skips test pads (exempt by rule; the re-placement put TP7 first)

Co-Authored-By: Claude Opus 5.5 <noreply@anthropic.com>
Claude-Session: https://claude.ai/code/session_01Wg997D6KFs8bxoAH56jZZJ
Other:
- title: Pod board Rev F: Speaker driver and ear pad -> Pod board Rev G: Speaker driver and ear pad
Changed lines of the file:
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@@
 	(paper "A4")
 	(title_block
-		(title "Pod board Rev F: Speaker driver and ear pad")
+		(title "Pod board Rev G: Speaker driver and ear pad")
 		(date "2026-10-02")
-		(rev "F")
+		(rev "G")
 		(company "Stereo Ultrasound")
 		(comment 1 "Generated by hw/pod/sch.py from hw/pod/pod.net (gen.py). Do not edit by hand.")
@@
 		(on_board yes)
 		(dnp no)
-		(property "Reference" "#PWR078"
+		(property "Reference" "#PWR079"
 			(at 88.9 66.04 0)
 			(effects
@@
 			(project "pod"
 				(path "/46f56cb9-40b8-53c9-9ea1-5c731f397bba/0d146cbe-3b0c-5247-93c7-46dd075005f9"
-					(reference "#PWR078")
+					(reference "#PWR079")
 					(unit 1)
 				)
@@
 		(on_board yes)
 		(dnp no)
-		(property "Reference" "#PWR079"
+		(property "Reference" "#PWR080"
 			(at 177.8 66.04 0)
 			(effects
@@
 			(project "pod"
 				(path "/46f56cb9-40b8-53c9-9ea1-5c731f397bba/0d146cbe-3b0c-5247-93c7-46dd075005f9"
-					(reference "#PWR079")
+					(reference "#PWR080")
 					(unit 1)
 				)
@@
 		(on_board yes)
 		(dnp no)
-		(property "Reference" "#PWR080"
+		(property "Reference" "#PWR081"
 			(at 73.66 60.96 0)
 			(effects
@@
 			(project "pod"
 				(path "/46f56cb9-40b8-53c9-9ea1-5c731f397bba/0d146cbe-3b0c-5247-93c7-46dd075005f9"
-					(reference "#PWR080")
+					(reference "#PWR081")
 					(unit 1)
 				)
@@
 		(on_board yes)
 		(dnp no)
-		(property "Reference" "#PWR081"
+		(property "Reference" "#PWR082"
 			(at 73.66 91.44 0)
 			(effects
@@
 			(project "pod"
 				(path "/46f56cb9-40b8-53c9-9ea1-5c731f397bba/0d146cbe-3b0c-5247-93c7-46dd075005f9"
-					(reference "#PWR081")
+					(reference "#PWR082")
 					(unit 1)
 				)
@@
 		(on_board yes)
 		(dnp no)
-		(property "Reference" "#PWR082"
+		(property "Reference" "#PWR083"
 			(at 162.56 60.96 0)
 			(effects
@@
 			(project "pod"
 				(path "/46f56cb9-40b8-53c9-9ea1-5c731f397bba/0d146cbe-3b0c-5247-93c7-46dd075005f9"
-					(reference "#PWR082")
+					(reference "#PWR083")
 					(unit 1)
 				)
@@
 		(on_board yes)
 		(dnp no)
-		(property "Reference" "#PWR083"
+		(property "Reference" "#PWR084"
 			(at 162.56 91.44 0)
 			(effects
@@
 			(project "pod"
 				(path "/46f56cb9-40b8-53c9-9ea1-5c731f397bba/0d146cbe-3b0c-5247-93c7-46dd075005f9"
-					(reference "#PWR083")
+					(reference "#PWR084")
 					(unit 1)
 				)
@@
 		(on_board yes)
 		(dnp no)
-		(property "Reference" "#PWR084"
+		(property "Reference" "#PWR085"
 			(at 127 107.95 0)
 			(effects
@@
 			(project "pod"
 				(path "/46f56cb9-40b8-53c9-9ea1-5c731f397bba/0d146cbe-3b0c-5247-93c7-46dd075005f9"
-					(reference "#PWR084")
+					(reference "#PWR085")
 					(unit 1)
 				)
@@
 		(on_board yes)
 		(dnp no)
-		(property "Reference" "#PWR085"
+		(property "Reference" "#PWR086"
 			(at 154.94 120.65 0)
 			(effects
@@
 			(project "pod"
 				(path "/46f56cb9-40b8-53c9-9ea1-5c731f397bba/0d146cbe-3b0c-5247-93c7-46dd075005f9"
-					(reference "#PWR085")
+					(reference "#PWR086")
 					(unit 1)
 				)
@@
 		(on_board yes)
 		(dnp no)
-		(property "Reference" "#PWR086"
+		(property "Reference" "#PWR087"
 			(at 38.1 46.99 0)
 			(effects
@@
 			(project "pod"
 				(path "/46f56cb9-40b8-53c9-9ea1-5c731f397bba/0d146cbe-3b0c-5247-93c7-46dd075005f9"
-					(reference "#PWR086")
+					(reference "#PWR087")
 					(unit 1)
 				)
@@
 		(on_board yes)
 		(dnp no)
-		(property "Reference" "#PWR087"
+		(property "Reference" "#PWR088"
 			(at 38.1 54.61 0)
 			(effects
@@
 			(project "pod"
 				(path "/46f56cb9-40b8-53c9-9ea1-5c731f397bba/0d146cbe-3b0c-5247-93c7-46dd075005f9"
-					(reference "#PWR087")
+					(reference "#PWR088")
 					(unit 1)
 				)
@@
 		(on_board yes)
 		(dnp no)
-		(property "Reference" "#PWR088"
+		(property "Reference" "#PWR089"
 			(at 44.45 142.24 90)
 			(effects
@@
 			(project "pod"
 				(path "/46f56cb9-40b8-53c9-9ea1-5c731f397bba/0d146cbe-3b0c-5247-93c7-46dd075005f9"
-					(reference "#PWR088")
-					(unit 1)
-				)
+					(reference "#PWR089")
+					(unit 1)
+				)
