File: hw/pod/sch/pod.kicad_sch (KiCad schematic)
At the start: 0 parts

Commit message: Rev G (ECR-0017, owner O24): C8/C9 back to 10 V-rated 2.2 uF C107369 (ST DS13737 Rev 10 p.153); D6 TPD1E10B06 ESD at the exposed CC contact J12 (same part/BOM line as D5)
- gen.py Rev G: 53 placed parts, 30 BOM lines, ERC 0; bom_check identity + part_heights for C107369
- board re-placed + routed (D6 on B behind J12, one via): 694 tracks, 118 vias, 1 unconnected (I2C_SDA, router
  variance), DRC 19 courtyard + 1 clearance 0.0892 vs 0.09 mm (router rounding); Phase-2 board supersedes it
- schematic pages regenerated (D6 on the dock sheet, Rev G title): connectivity PASS, 195 memberships
- tracker: new relations R-SMPS-BOARD, R-CLOCK-BOARD, R-UI-BOARD (miniaturization MZG-15 blind spot); all reviewed,
  0 suspect / 0 stale; docs updated (sub-processing issue 1 closed, sub-dock-usb F15, reg-board route, 00-whole counts)
- interfaces.py self-test: the clamp-band victim skips test pads (exempt by rule; the re-placement put TP7 first)

Co-Authored-By: Claude Opus 5.5 <noreply@anthropic.com>
Claude-Session: https://claude.ai/code/session_01Wg997D6KFs8bxoAH56jZZJ
Other:
- title: Pod board Rev F: schematic (generated from gen.py) -> Pod board Rev G: schematic (generated from gen.py)
Changed lines of the file:
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@@
 	(paper "A4")
 	(title_block
-		(title "Pod board Rev F: schematic (generated from gen.py)")
+		(title "Pod board Rev G: schematic (generated from gen.py)")
 		(date "2026-10-02")
-		(rev "F")
+		(rev "G")
 		(company "Stereo Ultrasound")
 	)
