File: hw/pod/sch/power.kicad_sch (KiCad schematic)
At the start: 15 parts, among them J5 BAT+, J9 NTC, U3 BQ25180YBGR, U4 TPS7A2030PDQNR

Commit message: Rev G (ECR-0017, owner O24): C8/C9 back to 10 V-rated 2.2 uF C107369 (ST DS13737 Rev 10 p.153); D6 TPD1E10B06 ESD at the exposed CC contact J12 (same part/BOM line as D5)
- gen.py Rev G: 53 placed parts, 30 BOM lines, ERC 0; bom_check identity + part_heights for C107369
- board re-placed + routed (D6 on B behind J12, one via): 694 tracks, 118 vias, 1 unconnected (I2C_SDA, router
  variance), DRC 19 courtyard + 1 clearance 0.0892 vs 0.09 mm (router rounding); Phase-2 board supersedes it
- schematic pages regenerated (D6 on the dock sheet, Rev G title): connectivity PASS, 195 memberships
- tracker: new relations R-SMPS-BOARD, R-CLOCK-BOARD, R-UI-BOARD (miniaturization MZG-15 blind spot); all reviewed,
  0 suspect / 0 stale; docs updated (sub-processing issue 1 closed, sub-dock-usb F15, reg-board route, 00-whole counts)
- interfaces.py self-test: the clamp-band victim skips test pads (exempt by rule; the re-placement put TP7 first)

Co-Authored-By: Claude Opus 5.5 <noreply@anthropic.com>
Claude-Session: https://claude.ai/code/session_01Wg997D6KFs8bxoAH56jZZJ
Other:
- title: Pod board Rev F: Charger, battery, 3.0 V -> Pod board Rev G: Charger, battery, 3.0 V
Changed lines of the file:
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@@
 	(paper "A4")
 	(title_block
-		(title "Pod board Rev F: Charger, battery, 3.0 V")
+		(title "Pod board Rev G: Charger, battery, 3.0 V")
 		(date "2026-10-02")
-		(rev "F")
+		(rev "G")
 		(company "Stereo Ultrasound")
 		(comment 1 "Generated by hw/pod/sch.py from hw/pod/pod.net (gen.py). Do not edit by hand.")
@@
 		(on_board yes)
 		(dnp no)
-		(property "Reference" "#PWR011"
+		(property "Reference" "#PWR012"
 			(at 17.78 157.48 0)
 			(effects
@@
 			(project "pod"
 				(path "/46f56cb9-40b8-53c9-9ea1-5c731f397bba/4bc0e25a-c0da-5268-b5b3-ecda7bc65689"
-					(reference "#PWR011")
+					(reference "#PWR012")
 					(unit 1)
 				)
@@
 		(on_board yes)
 		(dnp no)
-		(property "Reference" "#FLG012"
+		(property "Reference" "#FLG013"
 			(at 17.78 157.48 0)
 			(effects
@@
 			(project "pod"
 				(path "/46f56cb9-40b8-53c9-9ea1-5c731f397bba/4bc0e25a-c0da-5268-b5b3-ecda7bc65689"
-					(reference "#FLG012")
+					(reference "#FLG013")
 					(unit 1)
 				)
@@
 		(on_board yes)
 		(dnp no)
-		(property "Reference" "#PWR013"
+		(property "Reference" "#PWR014"
 			(at 33.02 157.48 0)
 			(effects
@@
 			(project "pod"
 				(path "/46f56cb9-40b8-53c9-9ea1-5c731f397bba/4bc0e25a-c0da-5268-b5b3-ecda7bc65689"
-					(reference "#PWR013")
+					(reference "#PWR014")
 					(unit 1)
 				)
@@
 		(on_board yes)
 		(dnp no)
-		(property "Reference" "#FLG014"
+		(property "Reference" "#FLG015"
 			(at 33.02 157.48 0)
 			(effects
@@
 			(project "pod"
 				(path "/46f56cb9-40b8-53c9-9ea1-5c731f397bba/4bc0e25a-c0da-5268-b5b3-ecda7bc65689"
-					(reference "#FLG014")
+					(reference "#FLG015")
 					(unit 1)
 				)
@@
 		(on_board yes)
 		(dnp no)
-		(property "Reference" "#PWR015"
+		(property "Reference" "#PWR016"
 			(at 48.26 157.48 0)
 			(effects
@@
 			(project "pod"
 				(path "/46f56cb9-40b8-53c9-9ea1-5c731f397bba/4bc0e25a-c0da-5268-b5b3-ecda7bc65689"
-					(reference "#PWR015")
+					(reference "#PWR016")
 					(unit 1)
 				)
@@
 		(on_board yes)
 		(dnp no)
-		(property "Reference" "#FLG016"
+		(property "Reference" "#FLG017"
 			(at 48.26 157.48 0)
 			(effects
@@
 			(project "pod"
 				(path "/46f56cb9-40b8-53c9-9ea1-5c731f397bba/4bc0e25a-c0da-5268-b5b3-ecda7bc65689"
-					(reference "#FLG016")
+					(reference "#FLG017")
 					(unit 1)
 				)
@@
 		(on_board yes)
 		(dnp no)
-		(property "Reference" "#PWR017"
+		(property "Reference" "#PWR018"
 			(at 63.5 157.48 0)
 			(effects
@@
 			(project "pod"
 				(path "/46f56cb9-40b8-53c9-9ea1-5c731f397bba/4bc0e25a-c0da-5268-b5b3-ecda7bc65689"
-					(reference "#PWR017")
+					(reference "#PWR018")
 					(unit 1)
 				)
@@
 		(on_board yes)
 		(dnp no)
-		(property "Reference" "#FLG018"
+		(property "Reference" "#FLG019"
 			(at 63.5 157.48 0)
 			(effects
@@
 			(project "pod"
 				(path "/46f56cb9-40b8-53c9-9ea1-5c731f397bba/4bc0e25a-c0da-5268-b5b3-ecda7bc65689"
-					(reference "#FLG018")
+					(reference "#FLG019")
 					(unit 1)
 				)
@@
 		(on_board yes)
 		(dnp no)
-		(property "Reference" "#PWR019"
+		(property "Reference" "#PWR020"
 			(at 78.74 157.48 0)
 			(effects
@@
 			(project "pod"
 				(path "/46f56cb9-40b8-53c9-9ea1-5c731f397bba/4bc0e25a-c0da-5268-b5b3-ecda7bc65689"
-					(reference "#PWR019")
+					(reference "#PWR020")
 					(unit 1)
 				)
@@
 		(on_board yes)
 		(dnp no)
-		(property "Reference" "#FLG020"
+		(property "Reference" "#FLG021"
 			(at 78.74 157.48 0)
 			(effects
@@
 			(project "pod"
 				(path "/46f56cb9-40b8-53c9-9ea1-5c731f397bba/4bc0e25a-c0da-5268-b5b3-ecda7bc65689"
-					(reference "#FLG020")
+					(reference "#FLG021")
 					(unit 1)
 				)
@@
 		(on_board yes)
 		(dnp no)
-		(property "Reference" "#PWR021"
+		(property "Reference" "#PWR022"
 			(at 102.87 80.01 90)
 			(effects
@@
 			(project "pod"
 				(path "/46f56cb9-40b8-53c9-9ea1-5c731f397bba/4bc0e25a-c0da-5268-b5b3-ecda7bc65689"
-					(reference "#PWR021")
+					(reference "#PWR022")
 					(unit 1)
 				)
@@
 		(on_board yes)
 		(dnp no)
-		(property "Reference" "#PWR022"
+		(property "Reference" "#PWR023"
 			(at 38.1 85.09 0)
 			(effects
@@
 			(project "pod"
 				(path "/46f56cb9-40b8-53c9-9ea1-5c731f397bba/4bc0e25a-c0da-5268-b5b3-ecda7bc65689"
-					(reference "#PWR022")
+					(reference "#PWR023")
 					(unit 1)
 				)
@@
 		(on_board yes)
 		(dnp no)
-		(property "Reference" "#PWR023"
+		(property "Reference" "#PWR024"
 			(at 68.58 91.44 0)
 			(effects
@@
 			(project "pod"
 				(path "/46f56cb9-40b8-53c9-9ea1-5c731f397bba/4bc0e25a-c0da-5268-b5b3-ecda7bc65689"
-					(reference "#PWR023")
+					(reference "#PWR024")
 					(unit 1)
 				)
@@
 		(on_board yes)
 		(dnp no)
-		(property "Reference" "#PWR024"
+		(property "Reference" "#PWR025"
 			(at 116.84 60.96 0)
 			(effects
@@
 			(project "pod"
 				(path "/46f56cb9-40b8-53c9-9ea1-5c731f397bba/4bc0e25a-c0da-5268-b5b3-ecda7bc65689"
-					(reference "#PWR024")
+					(reference "#PWR025")
 					(unit 1)
 				)
@@
 		(on_board yes)
 		(dnp no)
-		(property "Reference" "#PWR025"
+		(property "Reference" "#PWR026"
 			(at 109.22 60.96 0)
 			(effects
@@
 			(project "pod"
 				(path "/46f56cb9-40b8-53c9-9ea1-5c731f397bba/4bc0e25a-c0da-5268-b5b3-ecda7bc65689"
-					(reference "#PWR025")
+					(reference "#PWR026")
 					(unit 1)
 				)
@@
 		(on_board yes)
 		(dnp no)
-		(property "Reference" "#PWR026"
+		(property "Reference" "#PWR027"
 			(at 116.84 88.9 0)
 			(effects
@@
 			(project "pod"
 				(path "/46f56cb9-40b8-53c9-9ea1-5c731f397bba/4bc0e25a-c0da-5268-b5b3-ecda7bc65689"
-					(reference "#PWR026")
+					(reference "#PWR027")
 					(unit 1)
 				)
@@
 		(on_board yes)
 		(dnp no)
-		(property "Reference" "#PWR027"
+		(property "Reference" "#PWR028"
 			(at 124.46 93.98 0)
 			(effects
@@
 			(project "pod"
 				(path "/46f56cb9-40b8-53c9-9ea1-5c731f397bba/4bc0e25a-c0da-5268-b5b3-ecda7bc65689"
-					(reference "#PWR027")
+					(reference "#PWR028")
 					(unit 1)
 				)
@@
 		(on_board yes)
 		(dnp no)
-		(property "Reference" "#PWR028"
+		(property "Reference" "#PWR029"
 			(at 153.67 83.82 90)
 			(effects
@@
 			(project "pod"
 				(path "/46f56cb9-40b8-53c9-9ea1-5c731f397bba/4bc0e25a-c0da-5268-b5b3-ecda7bc65689"
-					(reference "#PWR028")
+					(reference "#PWR029")
 					(unit 1)
 				)
@@
 		(on_board yes)
 		(dnp no)
-		(property "Reference" "#PWR029"
+		(property "Reference" "#PWR030"
 			(at 142.24 73.66 0)
 			(effects
@@
 			(project "pod"
 				(path "/46f56cb9-40b8-53c9-9ea1-5c731f397bba/4bc0e25a-c0da-5268-b5b3-ecda7bc65689"
-					(reference "#PWR029")
+					(reference "#PWR030")
 					(unit 1)
 				)
@@
 		(on_board yes)
 		(dnp no)
-		(property "Reference" "#PWR030"
+		(property "Reference" "#PWR031"
 			(at 160.02 88.9 0)
 			(effects
@@
 			(project "pod"
 				(path "/46f56cb9-40b8-53c9-9ea1-5c731f397bba/4bc0e25a-c0da-5268-b5b3-ecda7bc65689"
-					(reference "#PWR030")
+					(reference "#PWR031")
 					(unit 1)
 				)
@@
 		(on_board yes)
 		(dnp no)
-		(property "Reference" "#PWR031"
+		(property "Reference" "#PWR032"
 			(at 176.53 78.74 0)
 			(effects
@@
 			(project "pod"
 				(path "/46f56cb9-40b8-53c9-9ea1-5c731f397bba/4bc0e25a-c0da-5268-b5b3-ecda7bc65689"
-					(reference "#PWR031")
+					(reference "#PWR032")
 					(unit 1)
 				)
@@
 		(on_board yes)
 		(dnp no)
-		(property "Reference" "#PWR032"
+		(property "Reference" "#PWR033"
 			(at 30.48 129.54 0)
 			(effects
@@
 			(project "pod"
 				(path "/46f56cb9-40b8-53c9-9ea1-5c731f397bba/4bc0e25a-c0da-5268-b5b3-ecda7bc65689"
-					(reference "#PWR032")
+					(reference "#PWR033")
 					(unit 1)
 				)
@@
 		(on_board yes)
 		(dnp no)
-		(property "Reference" "#PWR033"
+		(property "Reference" "#PWR034"
 			(at 20.32 129.54 0)
 			(effects
@@
 			(project "pod"
 				(path "/46f56cb9-40b8-53c9-9ea1-5c731f397bba/4bc0e25a-c0da-5268-b5b3-ecda7bc65689"
-					(reference "#PWR033")
+					(reference "#PWR034")
 					(unit 1)
 				)
@@
 		(on_board yes)
 		(dnp no)
-		(property "Reference" "#PWR034"
+		(property "Reference" "#PWR035"
 			(at 74.93 77.47 90)
 			(effects
@@
 			(project "pod"
 				(path "/46f56cb9-40b8-53c9-9ea1-5c731f397bba/4bc0e25a-c0da-5268-b5b3-ecda7bc65689"
-					(reference "#PWR034")
+					(reference "#PWR035")
 					(unit 1)
 				)
@@
 		(on_board yes)
 		(dnp no)
-		(property "Reference" "#PWR040"
+		(property "Reference" "#PWR041"
 			(at 127 77.47 90)
 			(effects
@@
 			(project "pod"
 				(path "/46f56cb9-40b8-53c9-9ea1-5c731f397bba/4bc0e25a-c0da-5268-b5b3-ecda7bc65689"
-					(reference "#PWR040")
+					(reference "#PWR041")
 					(unit 1)
 				)
@@
 		(on_board yes)
 		(dnp no)
-		(property "Reference" "#PWR041"
+		(property "Reference" "#PWR042"
 			(at 38.1 72.39 0)
 			(effects
@@
 			(project "pod"
 				(path "/46f56cb9-40b8-53c9-9ea1-5c731f397bba/4bc0e25a-c0da-5268-b5b3-ecda7bc65689"
-					(reference "#PWR041")
+					(reference "#PWR042")
 					(unit 1)
 				)
