File: hw/pod/k4/out/P/routed.kicad_pcb (KiCad board)
At the start: 6 copper layers, 15.5 x 12 mm, 37 parts, among them J1 TestPoint_Pad_D1.0mm, J2 TestPoint_Pad_D1.0mm, J21 CONN-SMD_BM28B0.6-30DP-2-0.35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, Q1 Nexperia_SOT1216_DFN1010B-6, Q2 Nexperia_SOT1216_DFN1010B-6, U1 QFN-48-1EP_7x7mm_P0.5mm_EP5.6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, Y1 Crystal_SMD_2012-2Pin_2.0x1.2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

Commit message: K4 re-place/route after 9ec84ae: P and M at L 15.5, plain kicad-cli DRC 0 errors / 0 unconnected both; route_net3d GRID env; pin-contract + ECR-0020 + backlog (C9/C17 datasheet check still open)
Co-Authored-By: Claude Opus 5.5 <noreply@anthropic.com>
Claude-Session: https://claude.ai/code/session_01Wg997D6KFs8bxoAH56jZZJ
Parts:
- C9: value C_0402_1005Metric -> C_0201_0603Metric; footprint C_0402_1005Metric -> C_0201_0603Metric
- J2: moved to B.Cu
- moved J2 2.40 mm to (2.00, 1.20), turned to 180 degrees
Connections:
- J21 pad 1: GND -> MIC_VDD
- J21 pad 11: USB_DP -> USB_DM
- J21 pad 13: USB_DM -> USB_DP
- J21 pad 15: GND -> +3V0
- J21 pad 17: +3V0 -> GND
- J21 pad 18: +3V0 -> GND
- J21 pad 19: +3V0 -> LED_K
- J21 pad 21: GND -> MIC_DATA
- J21 pad 22: TS -> GND
- J21 pad 23: I2C_SCL -> CHG_INT
- J21 pad 25: I2C_SDA -> BTN
- J21 pad 26: CHG_INT -> GND
- J21 pad 28: VBAT_SENSE -> GND
- J21 pad 29: BTN -> TS
- J21 pad 30: LED_K -> +3V0
- J21 pad 31: (no net) -> +3V0
- J21 pad 32: (no net) -> +3V0
- J21 pad 33: (no net) -> +3V0
- J21 pad 34: (no net) -> +3V0
- J21 pad 5: GND -> VBAT_SENSE
- J21 pad 6: MIC_VDD -> GND
- J21 pad 7: MIC_DATA -> I2C_SCL
- J21 pad 9: GND -> I2C_SDA
Routing:
- net MIC_VDD: track 13.4 -> 3.55 mm, vias 2 -> 1
- net I2C_SCL: track 14.0 -> 5.23 mm, vias 2 -> 1
- net VBAT_SENSE: track 4.00 -> 11.9 mm
- net I2C_SDA: track 12.6 -> 5.32 mm, vias 2 -> 1
- net LED_K: track 12.6 -> 6.40 mm, vias 2 -> 1
- net TS: track 7.75 -> 2.32 mm
- net MIC_CLK: track 17.3 -> 12.5 mm
- net MIC_DATA: track 5.25 -> 9.98 mm, vias 1 -> 2
- net USB_DP: track 9.24 -> 4.65 mm, vias 2 -> 1
- net CHG_INT: track 14.5 -> 10.4 mm
- net USB_DM: track 8.16 -> 4.57 mm, vias 2 -> 1
- net +3V0: track 31.7 -> 34.8 mm, vias 18 -> 17
- net GB_P: track 20.0 -> 17.2 mm, vias 5 -> 6
- net BTN: track 5.03 -> 2.48 mm, vias 2 -> 1
- net OUT_A: track 10.9 -> 13.3 mm
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